Commit message: first urdf file simulated

File: robocon27_simulation/urdf/due_wheel.urdf (robot description, URDF)
Before this commit: robot due_wheel, 5 links, 4 joints
Links:
- link backduewheels: mass 1 -> 0.25
- link backnormalwheel: mass 1 -> 0.25; geometry collision cylinder length=0.6647 radius=0.0636; visual mesh filename=package://robocon27_simulation/meshes/backnormalwheel.STL
- link base_link: mass 25 -> 30
- link frontdue: mass 1 -> 0.25
- link frontnormalwheels: mass 1 -> 0.25; geometry collision cylinder length=0.6647 radius=0.0636; visual mesh filename=package://robocon27_simulation/meshes/frontnormalwheels.STL
Joints:
- joint back_due_joint: limit (none) -> effort=45 velocity=30; origin xyz=1.0391 -1.4441 1.0284 rpy=1.5708 0.39092 0 -> xyz=0.25710 0.08490 0.07540 rpy=1.5708 0.39092 0
- joint back_normal_joint: limit (none) -> effort=45 velocity=30; origin xyz=0.97994 -1.1967 1.0165 rpy=1.5708 0.31067 0 -> xyz=0.19794 0.33230 0.06350 rpy=1.5708 0.31067 0
- joint front_due_joint: limit (none) -> effort=45 velocity=30; origin xyz=0.64914 -1.3091 1.0253 rpy=1.5708 0.43155 0 -> xyz=-0.13286 0.21990 0.07230 rpy=1.5708 0.43155 0
- joint front_normal_joint: limit (none) -> effort=45 velocity=30; origin xyz=0.57614 -1.1967 1.0165 rpy=-1.5708 1.5512 -3.1416 -> xyz=-0.20586 0.33230 0.06350 rpy=-1.5708 1.5512 -3.1416

Commit message: fix new urdf ff file

File: robocon27_simulation/urdf/due_wheel.urdf (robot description, URDF)
Before this commit: robot due_wheel, 5 links, 4 joints
Links:
- removed link backduewheels
- removed link backnormalwheel
- removed link frontdue
- removed link frontnormalwheels
- added link back_due, mass 2; collision mesh filename=package://robocon27_simulation/meshes/backduewheels.STL; visual mesh filename=package://robocon27_simulation/meshes/backduewheels.STL
- added link front_due, mass 2; collision mesh filename=package://robocon27_simulation/meshes/frontdue.STL; visual mesh filename=package://robocon27_simulation/meshes/frontdue.STL
- added link front_left_wheel, mass 1; collision cylinder length=0.0687 radius=0.0635; visual mesh filename=package://robocon27_simulation/meshes/1normalwheelf.STL
- added link front_right_wheel, mass 1; collision cylinder length=0.0687 radius=0.0635; visual mesh filename=package://robocon27_simulation/meshes/2normalwheelf.STL
- added link rear_left_wheel, mass 1; collision cylinder length=0.0687 radius=0.0635; visual mesh filename=package://robocon27_simulation/meshes/1normalwheelb.STL
- added link rear_right_wheel, mass 1; collision cylinder length=0.0687 radius=0.0635; visual mesh filename=package://robocon27_simulation/meshes/2wheelnormalbac.STL
- link base_link: mass 30 -> 22
Joints:
- removed joint back_normal_joint
- removed joint front_normal_joint
- added joint front_left_wheel_joint: type continuous, parent base_link, child front_left_wheel, origin xyz=0.205777 0.297999 -0.27 rpy=0 0 0, axis 0 1 0, limit effort=30 velocity=60
- added joint front_right_wheel_joint: type continuous, parent base_link, child front_right_wheel, origin xyz=0.205777 -0.298001 -0.27 rpy=0 0 0, axis 0 1 0, limit effort=30 velocity=60
- added joint rear_left_wheel_joint: type continuous, parent base_link, child rear_left_wheel, origin xyz=-0.198022 0.297999 -0.27 rpy=0 0 0, axis 0 1 0, limit effort=30 velocity=60
- added joint rear_right_wheel_joint: type continuous, parent base_link, child rear_right_wheel, origin xyz=-0.198022 -0.298001 -0.27 rpy=0 0 0, axis 0 1 0, limit effort=30 velocity=60
- joint back_due_joint: axis 0 0 1 -> 0 1 0; child backduewheels -> back_due; limit effort=45 velocity=30 -> effort=30 velocity=30; origin xyz=0.25710 0.08490 0.07540 rpy=1.5708 0.39092 0 -> xyz=-0.257216 -0.085 -0.258144 rpy=0 0 0
- joint front_due_joint: axis 0 0 1 -> 0 1 0; child frontdue -> front_due; limit effort=45 velocity=30 -> effort=30 velocity=30; origin xyz=-0.13286 0.21990 0.07230 rpy=1.5708 0.43155 0 -> xyz=0.132775 -0.22 -0.261273 rpy=0 0 0

Commit message: fix teleop script and re-orient due joint so the robot doesnt have to go up the stairs backwards

File: robocon27_simulation/urdf/due_wheel.urdf (robot description, URDF)
Before this commit: robot due_wheel, 7 links, 6 joints
Links:
- link base_link: mass 22 -> 20
Joints:
- joint back_due_joint: origin xyz=-0.257216 -0.085 -0.258144 rpy=0 0 0 -> xyz=-0.257216 0.085 -0.258144 rpy=0 0 3.141593
- joint front_due_joint: origin xyz=0.132775 -0.22 -0.261273 rpy=0 0 0 -> xyz=0.132775 0.22 -0.261273 rpy=0 0 3.141593
